File: KicadJE-EuroPowerSupply.kicad_pcb (KiCad board)
At the start: 2 copper layers, 100 x 100 mm, 97 parts, among them J101 Laptop Power, J102 +-15V thru, J103 +-12v out, J104 +5V out, J105 Laptop Power Out, J106 FrontInterConnVin, J107 BaseInterConnVin, J108 FrontInterConnVout, J109 BaseInterConnVout, P101 Doepfer_Power_10pin, P102 Doepfer_Power_16pin, P105 Doepfer_Power_10pin, P106 Doepfer_Power_16pin, Q201 TIP41, Q202 TIP41, Q203 TIP42, SW101 SW_SPDT, U201 LM7812_TO220, U202 LM7805_TO220, U203 Step Down Module +15 to 7v - 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, U204 LM7912_TO220, U205 XL6009 Module DCDC 19 to 30v, U206 TL071, U207 LM78M05_TO252, U208 LM78M12_TO252, U209 MC79M12_TO252, U210 MT3608 Module DCDC 19 to 28v

Commit message: Initial Route
Parts:
- added R209: 0r25, Resistor_THT:R_Axial_DIN0204_L3.6mm_D1.6mm_P5.08mm_Vertical, F.Cu at (165.8, 104.9)
- added R210: 0r25, Resistor_THT:R_Axial_DIN0204_L3.6mm_D1.6mm_P5.08mm_Vertical, F.Cu at (153.2, 123.0)
- added R211: 0r25, Resistor_THT:R_Axial_DIN0204_L3.6mm_D1.6mm_P5.08mm_Vertical, F.Cu at (169.8, 104.9)
- added R212: 0r25, Resistor_THT:R_Axial_DIN0204_L3.6mm_D1.6mm_P5.08mm_Vertical, F.Cu at (157.0, 123.0)
- added R213: 0r25, Resistor_THT:R_Axial_DIN0204_L3.6mm_D1.6mm_P5.08mm_Vertical, F.Cu at (173.3, 104.9)
- added R214: 0r25, Resistor_THT:R_Axial_DIN0204_L3.6mm_D1.6mm_P5.08mm_Vertical, F.Cu at (177.0, 104.9)
- C101, C204, C207: moved to B.Cu
- D206, R205: moved to F.Cu
- J106, J107: footprint AJ-Dropbox-Kicad:BoardConnector2x2.54x10mm2pin -> AJ-Dropbox-Kicad:BoardConnector2x2.54x10mm4pin
- moved C101 39.4 mm to (132.8, 82.5), turned to 270 degrees
- moved R202 24.9 mm to (180.0, 71.2)
- moved R206 23.5 mm to (181.5, 77.5)
- moved C210 22.4 mm to (178.8, 86.5)
- moved Q202 21.9 mm to (184.8, 73.2)
- moved C203 21.8 mm to (178.8, 68.5)
- moved C217 21.8 mm to (182.5, 69.5)
- moved R208 21.8 mm to (180.0, 83.4)
- moved C220 20.3 mm to (185.5, 85.5)
- moved Q203 20.3 mm to (182.8, 81.8)
- moved C212 16.1 mm to (174.0, 110.2), turned to 0 degrees
- moved D206 14.8 mm to (189.0, 56.2), turned to 270 degrees
- moved U206 12.0 mm to (165.0, 81.5)
- moved C218 11.9 mm to (160.3, 87.8)
- moved R207 11.9 mm to (162.3, 87.8)
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Routing:
- net -12V: track 37.4 -> 194.1 mm, vias 2 -> 11
- net +12V: track 139.0 -> 258.8 mm, vias 3 -> 28
- net +5V: track 64.0 -> 181.1 mm, vias 2 -> 14
- net Vin+15: track 0.00 -> 100.1 mm, vias 0 -> 5
- net GND: track 16.8 -> 115.6 mm, vias 18 -> 33
- net Vin-15: track 0.00 -> 88.5 mm
- net DCDC+: track 0.00 -> 73.5 mm, vias 0 -> 2
- net Vin-Neg19: track 22.5 -> 80.9 mm, vias 0 -> 4
- net Vin-Pos19: track 27.6 -> 76.2 mm
- net -15V: track 0.00 -> 44.3 mm, vias 0 -> 7
- net +7.5V: track 0.00 -> 41.3 mm, vias 0 -> 2
- net CV: track 0.00 -> 23.8 mm, vias 0 -> 2
- net Gate: track 0.00 -> 22.3 mm, vias 0 -> 2
- net +15V: track 0.00 -> 18.8 mm
- net Net-(C216-Pad2): track 0.00 -> 17.5 mm
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- added copper zone on B.Cu, net /DCSleeve
- added copper zone on F.Cu, net Net-(J101-Pad1)
- added copper zone on B.Cu, net Vin-Neg19
- added copper zone on F.Cu, net Vin-Pos19
- added copper zone on B.Cu, net VinGND
Other:
- board text added: "+19"
- board text added: "-19"

Commit message: Update KicadJE-EuroPowerSupply.kicad_pcb
Parts:
- added G***: LOGO, AJ:Johansen_engineering_logo_20mm, F.Cu at (137.6, 65.0)
- added G***: LOGO, AJ:Johansen_engineering_logo_25mm_front_neg5, B.Cu at (102.6, 139.2)
- added G***: LOGO, AJ:Johansen_engineering_logo_25mm_front_neg5, F.Cu at (161.0, 58.2)
- added G***: LOGO, AJ:Johansen_engineering_logo_25mm_front_neg5, B.Cu at (171.6, 125.4)
Other:
- board text added: "+12 +5 GND -12"

Commit message: DRC
Parts:
- U203: value Step Down Module +15 to 7v - MP2307 -> +15 to 7v - MP2307
- moved G*** 0.36 mm to (102.3, 139.0)
Routing:
- net GND: track 115.6 -> 121.5 mm, vias 33 -> 32
- net Net-(D104-Pad1): track 0.00 -> 2.97 mm
Other:
- board text added: "+15V"
- board text added: "+7V"
- board text added: "-15V"
- board text added: "DCDC In+"
- board text added: "DCDC In-"
- board text added: "DCDC+"
- board text added: "DCDC-"
- board text added: "GND"
- board text added: "VGND"

Commit message: faceplate text
Other:
- board text added: "+"
- board text added: "-"
- board text added: "gnd"
Changed lines of the file:
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@@
   (general
     (thickness 1.6)
-    (drawings 131)
+    (drawings 135)
     (tracks 690)
     (zones 0)
@@
     (descr "Barrel Jack, 2.0mm ID, 5.5mm OD, 24V, 8A, no switch, https://www.cui.com/product/resource/pj-063ah.pdf")
     (tags "barrel jack cui dc power")
-    (fp_text reference J105 (at 0 -2.3 180) (layer F.SilkS)
+    (fp_text reference J105 (at 0 3.6 180) (layer F.SilkS)
       (effects (font (size 1 1) (thickness 0.15)))
     )
-    (fp_text value "Laptop Power Out" (at 0 13 180) (layer F.Fab)
+    (fp_text value "Laptop Power Out" (at -0.2 -2.6 180) (layer F.SilkS)
       (effects (font (size 1 1) (thickness 0.15)))
     )
@@
     (at 122.2 129.07 270)
     (attr smd)
-    (fp_text reference J109 (at 0 6.15 270) (layer F.SilkS)
+    (fp_text reference J109 (at 2.83 4.1 270) (layer F.SilkS)
       (effects (font (size 1 1) (thickness 0.15)))
     )
@@
     (tags "Diode Mini-MELF Handsoldering")
     (attr smd)
-    (fp_text reference D102 (at 0 -1.75 90) (layer F.SilkS)
+    (fp_text reference D102 (at -2.75 -1.7 90) (layer F.SilkS)
       (effects (font (size 1 1) (thickness 0.15)))
     )
-    (fp_text value 27v (at 0 1.75 90) (layer F.Fab)
+    (fp_text value 27v (at -3.15 -3.05 90) (layer F.SilkS)
       (effects (font (size 1 1) (thickness 0.15)))
     )
@@
     (descr "LED, diameter 5.0mm, 2 pins, http://cdn-reichelt.de/documents/datenblatt/A500/LL-504BC2E-009.pdf")
     (tags "LED diameter 5.0mm 2 pins")
-    (fp_text reference D105 (at 1.27 -3.96) (layer F.SilkS)
+    (fp_text reference D105 (at -3.85 -2.65) (layer F.SilkS)
       (effects (font (size 1 1) (thickness 0.15)))
     )
@@
     (descr "LED, diameter 5.0mm, 2 pins, http://cdn-reichelt.de/documents/datenblatt/A500/LL-504BC2E-009.pdf")
     (tags "LED diameter 5.0mm 2 pins")
-    (fp_text reference D106 (at 1.27 -3.96) (layer F.SilkS)
+    (fp_text reference D106 (at -3.9 -2.45) (layer F.SilkS)
       (effects (font (size 1 1) (thickness 0.15)))
     )
@@
     (tags "resistor handsolder")
     (attr smd)
-    (fp_text reference F101 (at 0 -2.65) (layer F.SilkS)
+    (fp_text reference F101 (at -6.6 -0.4) (layer F.SilkS)
       (effects (font (size 1 1) (thickness 0.15)))
     )
-    (fp_text value 750mA (at 0 2.65) (layer F.Fab)
+    (fp_text value 750mA (at -6 1.35) (layer F.SilkS)
       (effects (font (size 1 1) (thickness 0.15)))
     )
@@
       (effects (font (size 1 1) (thickness 0.15)))
     )
-    (fp_text value 10r (at 0 1.65 90) (layer F.Fab)
+    (fp_text value 10r (at -0.7 -3.2 90) (layer F.SilkS)
       (effects (font (size 1 1) (thickness 0.15)))
     )
@@
     (tags "resistor handsolder")
     (attr smd)
-    (fp_text reference R102 (at 0 -1.65 270) (layer F.SilkS)
+    (fp_text reference R102 (at -0.05 -2.15 270) (layer F.SilkS)
       (effects (font (size 1 1) (thickness 0.15)))
     )
-    (fp_text value 10k (at 0 1.65 270) (layer F.Fab)
+    (fp_text value 10k (at -0.7 2.15 270) (layer F.SilkS)
       (effects (font (size 1 1) (thickness 0.15)))
     )
@@
       (effects (font (size 1 1) (thickness 0.15)))
     )
-    (fp_text value 4k7 (at 0 1.65) (layer F.Fab)
+    (fp_text value 4k7 (at 0 1.65) (layer F.SilkS)
       (effects (font (size 1 1) (thickness 0.15)))
     )
@@
       (effects (font (size 1 1) (thickness 0.15)))
     )
-    (fp_text value 1k5 (at 0 1.65) (layer F.Fab)
+    (fp_text value 1k5 (at 5 0.05) (layer F.SilkS)
       (effects (font (size 1 1) (thickness 0.15)))
     )
@@
       (effects (font (size 1 1) (thickness 0.15)))
     )
-    (fp_text value 4k7 (at 0 1.65) (layer F.Fab)
+    (fp_text value 4k7 (at 3.325 0.1) (layer F.SilkS)
       (effects (font (size 1 1) (thickness 0.15)))
     )
@@
     (descr "Varistor, diameter 12mm, width 4.8mm, pitch 7.5mm")
     (tags "varistor SIOV")
-    (fp_text reference RV101 (at 3.75 4.425 90) (layer F.SilkS)
+    (fp_text reference RV101 (at 0.6 2.3 90) (layer F.SilkS)
       (effects (font (size 1 1) (thickness 0.15)))
     )
@@
   (module AJ-Dropbox-Kicad:SP1MS1 (layer F.Cu)
     (at 110 78)
-    (fp_text reference SW101 (at -2.4 1.8) (layer F.SilkS)
+    (fp_text reference SW101 (at 0.05 2.3) (layer F.SilkS)
       (effects (font (size 1 1) (thickness 0.15)))
     )
@@
     (tags "test point THT pad")
     (attr virtual)
-    (fp_text reference TP101 (at 0 -1.998) (layer F.SilkS)
+    (fp_text reference TP101 (at -5.6 5.7) (layer F.SilkS)
       (effects (font (size 1 1) (thickness 0.15)))
     )
-    (fp_text value "RED Sleeve" (at 0 2.05) (layer F.Fab)
+    (fp_text value "RED Sleeve" (at -0.55 2.3) (layer F.Fab)
       (effects (font (size 1 1) (thickness 0.15)))
     )
@@
     (tags "mounting hole 6.4mm m6 iso14580")
     (attr virtual)
-    (fp_text reference TP102 (at 0 -6) (layer F.SilkS)
+    (fp_text reference TP102 (at 0.1 -0.1) (layer F.SilkS)
       (effects (font (size 1 1) (thickness 0.15)))
     )
-    (fp_text value "RED Banana" (at 0 6) (layer F.Fab)
+    (fp_text value "RED Banana" (at 0 6) (layer F.SilkS)
       (effects (font (size 1 1) (thickness 0.15)))
     )
@@
     (tags "test point THT pad")
     (attr virtual)
-    (fp_text reference TP103 (at 0 -1.998) (layer F.SilkS)
+    (fp_text reference TP103 (at -5.3 1.7) (layer F.SilkS)
       (effects (font (size 1 1) (thickness 0.15)))
     )
@@
     (tags "mounting hole 6.4mm m6 iso14580")
     (attr virtual)
-    (fp_text reference TP104 (at 0 -6) (layer F.SilkS)
+    (fp_text reference TP104 (at 0 0.1) (layer F.SilkS)
       (effects (font (size 1 1) (thickness 0.15)))
     )
-    (fp_text value "BLUE Banana" (at 0 6) (layer F.Fab)
+    (fp_text value "BLUE Banana" (at -1.25 -6.05) (layer F.SilkS)
       (effects (font (size 1 1) (thickness 0.15)))
     )
@@
     (tags "test point THT pad")
     (attr virtual)
-    (fp_text reference TP105 (at 0 -1.998) (layer F.SilkS)
+    (fp_text reference TP105 (at -5.4 1.7) (layer F.SilkS)
       (effects (font (size 1 1) (thickness 0.15)))
     )
@@
     (tags "mounting hole 6.4mm m6 iso14580")
     (attr virtual)
-    (fp_text reference TP106 (at 0 -6) (layer F.SilkS)
+    (fp_text reference TP106 (at 0.25 -1.15) (layer F.SilkS)
       (effects (font (size 1 1) (thickness 0.15)))
     )
-    (fp_text value "BLACK Banana" (at 0 6) (layer F.Fab)
+    (fp_text value "BLACK Banana" (at 0 6) (layer F.SilkS)
       (effects (font (size 1 1) (thickness 0.15)))
     )
@@
     (tags "test point THT pad")
     (attr virtual)
-    (fp_text reference TP107 (at 0 -1.998) (layer F.SilkS)
+    (fp_text reference TP107 (at -5.75 5.5) (layer F.SilkS)
       (effects (font (size 1 1) (thickness 0.15)))
     )
@@
     (tags "mounting hole 6.4mm m6 iso14580")
     (attr virtual)
-    (fp_text reference TP108 (at 0 -6) (layer F.SilkS)
+    (fp_text reference TP108 (at 0.1 -1.3) (layer F.SilkS)
       (effects (font (size 1 1) (thickness 0.15)))
     )
-    (fp_text value "RED Banana" (at 0 6) (layer F.Fab)
+    (fp_text value "RED Banana" (at 0 6) (layer F.SilkS)
       (effects (font (size 1 1) (thickness 0.15)))
     )
@@
     (descr "Barrel Jack, 2.0mm ID, 5.5mm OD, 24V, 8A, no switch, https://www.cui.com/product/resource/pj-063ah.pdf")
     (tags "barrel jack cui dc power")
-    (fp_text reference J101 (at 0 -2.3 180) (layer F.SilkS)
+    (fp_text reference J101 (at 0.1 3.05 180) (layer F.SilkS)
       (effects (font (size 1 1) (thickness 0.15)))
     )
-    (fp_text value "Laptop Power" (at 0 13 180) (layer F.Fab)
+    (fp_text value "Laptop Power" (at 3.65 -2.05 180) (layer F.SilkS)
       (effects (font (size 1 1) (thickness 0.15)))
     )
@@
       (xy 7.7216 2.1336)) (layer B.SilkS) (width 0.01))
   )
+  (gr_text - (at 126.35 142.45) (layer F.SilkS)
+    (effects (font (size 1 1) (thickness 0.25)))
+  )
+  (gr_text gnd (at 134.25 142.35) (layer F.SilkS)
+    (effects (font (size 1 1) (thickness 0.25)))
+  )
+  (gr_text + (at 134.1 112.35) (layer F.SilkS)
+    (effects (font (size 1 1) (thickness 0.25)))
+  )
+  (gr_text + (at 133.55 96.85) (layer F.SilkS)
+    (effects (font (size 1 1) (thickness 0.25)))
+  )
   (gr_text VGND (at 159.3 102.5) (layer F.SilkS)
